Commit message: 已适配h30，未进行精细校准

File: agribot_ws/install/turn_on_32chassis/share/turn_on_32chassis/urdf/urdf/mini_4wd_robot.urdf.xacro (robot description, xacro)
@@ -50,4 +50,12 @@
             </collision>
         </link>
+        <!-- H30 IMU mounting frame.
+             Replace xyz/rpy with the measured extrinsics of the sensor. -->
+        <link name="gyro_link" />
+        <joint name="h30_joint" type="fixed">
+            <origin xyz="0.03163 0.05 0.065" rpy="0 0 0" />
+            <parent link="base_link" />
+            <child link="gyro_link" />
+        </joint>
         <link
             name="lf_wheel_link">

Commit message: 完成雷达、h30、底盘的合成

File: agribot_ws/install/turn_on_32chassis/share/turn_on_32chassis/urdf/urdf/mini_4wd_robot.urdf.xacro (robot description, xacro)
@@ -52,7 +52,19 @@
         <!-- H30 IMU mounting frame.
              Replace xyz/rpy with the measured extrinsics of the sensor. -->
-        <link name="gyro_link" />
+        <!-- Yesense H30: 24.5 mm × 24.5 mm × 14.5 mm.
+             The gyro_link origin is the geometric centre of the enclosure. -->
+        <link name="gyro_link">
+            <visual>
+                <origin xyz="0 0 0" rpy="0 0 0" />
+                <geometry>
+                    <box size="0.0245 0.0245 0.0145" />
+                </geometry>
+                <material name="h30_enclosure">
+                    <color rgba="0.15 0.45 0.95 0.75" />
+                </material>
+            </visual>
+        </link>
         <joint name="h30_joint" type="fixed">
-            <origin xyz="0.03163 0.05 0.065" rpy="0 0 0" />
+            <origin xyz="0.047 0.043 0.060" rpy="0 0 0" />
             <parent link="base_link" />
             <child link="gyro_link" />
@@ -271,5 +283,5 @@
         </joint>
         <!-- laser -->
-         <!-- <link
+        <link
             name="laser_link">
             <inertial>
@@ -290,8 +302,8 @@
                 <origin
                     xyz="0 0 0"
-                    rpy="0 0 0" />
-                <geometry>
-                    <mesh
-                        filename="package://turn_on_32chassis/urdf/meshes/mini_4wd_robot_meshes/laser.STL" />
+                    rpy="0 3.14159265358979 0" />
+                <geometry>
+                    <mesh
+                        filename="package://turn_on_32chassis/urdf/meshes/mid-360-asm.stl" />
                 </geometry>
                 <material
@@ -304,8 +316,8 @@
                 <origin
                     xyz="0 0 0"
-                    rpy="0 0 0" />
-                <geometry>
-                    <mesh
-                        filename="package://turn_on_32chassis/urdf/meshes/mini_4wd_robot_meshes/laser.STL" />
+                    rpy="0 3.14159265358979 0" />
+                <geometry>
+                    <mesh
+                        filename="package://turn_on_32chassis/urdf/meshes/mid-360-asm.stl" />
                 </geometry>
             </collision>
@@ -315,6 +327,6 @@
             type="fixed">
             <origin
-                xyz="0.0316310367407428 9.05810809801877E-05 0.09292418374143"
-                rpy="0 0 3.14159265358979" />
+                xyz="0.0316310367407428 9.05810809801877E-05 0.115"
+                rpy="0 0 0" />
             <parent
                 link="base_link" />
@@ -323,5 +335,5 @@
             <axis
                 xyz="0 0 0" />
-        </joint>  -->
+        </joint>
         <link
             name="controller_link">
