Commit message: 实现FAST-LIO+IMU+轮速融合里程计解决车轮原地打滑的问题

File: agribot_ws/install/turn_on_32chassis/share/turn_on_32chassis/urdf/urdf/agribot.urdf.xacro (robot description, xacro)
@@ -1,28 +1 @@
-<?xml version="1.0"?>
-<robot xmlns:xacro="http://www.ros.org/wiki/xacro" name="agribot">
-    <!-- 基础组件 base_link -->
-    <!-- <xacro:include filename="$(find agribot_simulation)/urdf/agribot/mini_4wd_robot.urdf.xacro" /> -->
-    <xacro:include filename="mini_4wd_robot.urdf.xacro" />
-    <!-- mid360雷达 -->
-    <!-- <xacro:include filename="$(find ros2_livox_simulation)/urdf/mid360.xacro" /> -->
-    <!-- Gazebo相关配置 -->
-    <!-- <xacro:include filename="$(find agribot_simulation)/urdf/agribot/agribot.gazebo.xacro" /> -->
-    <!-- ROS2 Control配置 -->
-    <!-- <xacro:include filename="$(find agribot_simulation)/urdf/agribot/agribot.ros2_control.xacro" /> -->
-    <!-- Gazebo传感器插件 -->
-    <!-- <xacro:include
-        filename="$(find agribot_simulation)/urdf/agribot/plugins/gazebo_sensor_plugin.xacro" /> -->
-    <!-- Gazebo控制插件 -->
-    <!-- <xacro:include filename="$(find
-    agribot_simulation)/urdf/agribot/plugins/gazebo_control_plugin.xacro"/> -->
-    <xacro:mini_4wd_robot_xacro />
-    <!-- <xacro:imu_xacro xyz="0 0 0" /> -->
-    <!-- <xacro:mid360 name="livox" parent="base_link" topic="mid360">
-        <origin xyz="0.1 0 0.1" rpy="0 0 0" />
-    </xacro:mid360> -->
-    <!-- <xacro:agribot_ros2_control /> -->
-    <!-- 使用gazebo传感器插件宏 -->
-    <!-- <xacro:gazebo_sensor_plugin /> -->
-    <!-- 使用gazebo_control_plugin宏
-    <xacro:gazebo_control_plugin /> -->
-</robot>
+/home/wheeltec/agribot/agribot_ws/src/turn_on_32chassis/urdf/urdf/agribot.urdf.xacro

File: agribot_ws/install/turn_on_32chassis/share/turn_on_32chassis/urdf/urdf/mini_4wd_robot.urdf.xacro (robot description, xacro)
@@ -1,446 +1 @@
-<?xml version="1.0"?>
-<robot xmlns:xacro="http://www.ros.org/wiki/xacro">
-    <!-- 声明base模块 -->
-    <xacro:macro name="mini_4wd_robot_xacro">
-        <!-- 添加虚拟根链接以解决KDL警告 -->
-        <link name="base_footprint" />
-        <joint name="base_joint" type="fixed">
-            <origin xyz="0 0 0" rpy="0 0 0" />
-            <parent link="base_footprint" />
-            <child link="base_link" />
-        </joint>
-        <link
-            name="base_link">
-            <inertial>
-                <origin
-                    xyz="-0.0128421829279015 -0.0198593937870083 0.00472064301055347"
-                    rpy="0 0 0" />
-                <mass
-                    value="0.619760484843179" />
-                <inertia
-                    ixx="0.00049908549476667"
-                    ixy="-1.7170206624065E-06"
-                    ixz="-4.24523881219841E-07"
-                    iyy="0.000746458274197243"
-                    iyz="-7.41976515459759E-07"
-                    izz="0.00114198658204837" />
-            </inertial>
-            <visual>
-                <origin
-                    xyz="0 0 0"
-                    rpy="0 0 0" />
-                <geometry>
-                    <mesh
-                        filename="package://turn_on_32chassis/urdf/meshes/mini_4wd_robot_meshes/base_link.STL" />
-                </geometry>
-                <material
-                    name="">
-                    <color
-                        rgba="0.741176470588235 0.901960784313726 0.956862745098039 1" />
-                </material>
-            </visual>
-            <collision>
-                <origin
-                    xyz="0 0 0"
-                    rpy="0 0 0" />
-                <geometry>
-                    <mesh
-                        filename="package://turn_on_32chassis/urdf/meshes/mini_4wd_robot_meshes/base_link.STL" />
-                </geometry>
-            </collision>
-        </link>
-        <!-- H30 IMU mounting frame.
-             Replace xyz/rpy with the measured extrinsics of the sensor. -->
-        <!-- Yesense H30: 24.5 mm × 24.5 mm × 14.5 mm.
-             The gyro_link origin is the geometric centre of the enclosure. -->
-        <link name="gyro_link">
-            <visual>
-                <origin xyz="0 0 0" rpy="0 0 0" />
-                <geometry>
-                    <box size="0.0245 0.0245 0.0145" />
-                </geometry>
-                <material name="h30_enclosure">
-                    <color rgba="0.15 0.45 0.95 0.75" />
-                </material>
-            </visual>
-        </link>
-        <joint name="h30_joint" type="fixed">
-            <origin xyz="0.047 0.043 0.060" rpy="0 0 0" />
-            <parent link="base_link" />
-            <child link="gyro_link" />
-        </joint>
-        <link
-            name="lf_wheel_link">
-            <inertial>
-                <origin
-                    xyz="-1.27712550672052E-07 -0.000325096094343197 2.97668804279116E-07"
-                    rpy="0 0 0" />
-                <mass
-                    value="0.0420381277202372" />
-                <inertia
-                    ixx="1.72190960888397E-05"
-                    ixy="2.03639273675061E-09"
-                    ixz="2.4149299899044E-09"
-                    iyy="2.97212421151102E-05"
-                    iyz="-2.15428671658865E-11"
-                    izz="1.72364765737453E-05" />
-            </inertial>
-            <visual>
-                <origin
-                    xyz="0 0 0"
-                    rpy="0 0 0" />
-                <geometry>
-                    <mesh
-                        filename="package://turn_on_32chassis/urdf/meshes/mini_4wd_robot_meshes/lf_wheel_link.STL" />
-                </geometry>
-                <material
-                    name="">
-                    <color
-                        rgba="1 1 1 1" />
-                </material>
-            </visual>
-            <collision>
-                <origin
-                    xyz="0 0 0"
-                    rpy="0 0 0" />
-                <geometry>
-                    <mesh
-                        filename="package://turn_on_32chassis/urdf/meshes/mini_4wd_robot_meshes/lf_wheel_link.STL" />
-                </geometry>
-            </collision>
-        </link>
-        <joint
-            name="lf_wheel_joint"
-            type="continuous">
-            <origin
-                xyz="0.0788866867829701 0.090902092708038 -0.0363"
-                rpy="0 0 0" />
-            <parent
-                link="base_link" />
-            <child
-                link="lf_wheel_link" />
-            <axis
-                xyz="0 1 0" />
-        </joint>
-        <link
-            name="lb_wheel_link">
-            <inertial>
-                <origin
-                    xyz="-1.28150099226731E-07 -0.000325096043508583 2.97625719625216E-07"
-                    rpy="0 0 0" />
-                <mass
-                    value="0.0420381286687321" />
-                <inertia
-                    ixx="1.72190959347134E-05"
-                    ixy="2.03643074352543E-09"
-                    ixz="2.41484184900578E-09"
-                    iyy="2.97212425394595E-05"
-                    iyz="-2.15391461481771E-11"
-                    izz="1.72364771579999E-05" />
-            </inertial>
-            <visual>
-                <origin
-                    xyz="0 0 0"
-                    rpy="0 0 0" />
-                <geometry>
-                    <mesh
-                        filename="package://turn_on_32chassis/urdf/meshes/mini_4wd_robot_meshes/lb_wheel_link.STL" />
-                </geometry>
-                <material
-                    name="">
-                    <color
-                        rgba="1 1 1 1" />
-                </material>
-            </visual>
-            <collision>
-                <origin
-                    xyz="0 0 0"
-                    rpy="0 0 0" />
-                <geometry>
-                    <mesh
-                        filename="package://turn_on_32chassis/urdf/meshes/mini_4wd_robot_meshes/lb_wheel_link.STL" />
-                </geometry>
-            </collision>
-        </link>
-        <joint
-            name="lb_wheel_joint"
-            type="continuous">
-            <origin
-                xyz="-0.0930133132170299 0.0909020927080386 -0.0363"
-                rpy="0 0 0" />
-            <parent
-                link="base_link" />
-            <child
-                link="lb_wheel_link" />
-            <axis
-                xyz="0 1 0" />
-        </joint>
-        <link
-            name="rb_wheel_link">
-            <inertial>
-                <origin
-                    xyz="1.28149403894051E-07 0.000325096047440132 2.97624308309707E-07"
-                    rpy="0 0 0" />
-                <mass
-                    value="0.0420381286421594" />
-                <inertia
-                    ixx="1.72190962340715E-05"
-                    ixy="2.03640106869117E-09"
-                    ixz="-2.41477994262437E-09"
-                    iyy="2.97212428073701E-05"
-                    iyz="2.15356782895359E-11"
-                    izz="1.72364771452533E-05" />
-            </inertial>
-            <visual>
-                <origin
-                    xyz="0 0 0"
-                    rpy="0 0 0" />
-                <geometry>
-                    <mesh
-                        filename="package://turn_on_32chassis/urdf/meshes/mini_4wd_robot_meshes/rb_wheel_link.STL" />
-                </geometry>
-                <material
-                    name="">
-                    <color
-                        rgba="1 1 1 1" />
-                </material>
-            </visual>
-            <collision>
-                <origin
-                    xyz="0 0 0"
-                    rpy="0 0 0" />
-                <geometry>
-                    <mesh
-                        filename="package://turn_on_32chassis/urdf/meshes/mini_4wd_robot_meshes/rb_wheel_link.STL" />
-                </geometry>
-            </collision>
-        </link>
-        <joint
-            name="rb_wheel_joint"
-            type="continuous">
-            <origin
-                xyz="-0.0930053132170305 -0.0907239072919614 -0.0363"
-                rpy="0 0 0" />
-            <parent
-                link="base_link" />
-            <child
-                link="rb_wheel_link" />
-            <axis
-                xyz="0 1 0" />
-        </joint>
-        <link
-            name="rf_wheel_link">
-            <inertial>
-                <origin
-                    xyz="1.27697581011558E-07 0.000325096090387209 2.97695706086287E-07"
-                    rpy="0 0 0" />
-                <mass
-                    value="0.0420381277503723" />
-                <inertia
-                    ixx="1.7219096206293E-05"
-                    ixy="2.03637766318229E-09"
-                    ixz="-2.41488182670862E-09"
-                    iyy="2.97212422221003E-05"
-                    iyz="2.153998885685E-11"
-                    izz="1.72364765727325E-05" />
-            </inertial>
-            <visual>
-                <origin
-                    xyz="0 0 0"
-                    rpy="0 0 0" />
-                <geometry>
-                    <mesh
-                        filename="package://turn_on_32chassis/urdf/meshes/mini_4wd_robot_meshes/rf_wheel_link.STL" />
-                </geometry>
-                <material
-                    name="">
-                    <color
-                        rgba="1 1 1 1" />
-                </material>
-            </visual>
-            <collision>
-                <origin
-                    xyz="0 0 0"
-                    rpy="0 0 0" />
-                <geometry>
-                    <mesh
-                        filename="package://turn_on_32chassis/urdf/meshes/mini_4wd_robot_meshes/rf_wheel_link.STL" />
-                </geometry>
-            </collision>
-        </link>
-        <joint
-            name="rf_wheel_joint"
-            type="continuous">
-            <origin
-                xyz="0.0788946867829695 -0.090723907291962 -0.0363"
-                rpy="0 0 0" />
-            <parent
-                link="base_link" />
-            <child
-                link="rf_wheel_link" />
-            <axis
-                xyz="0 1 0" />
-        </joint>
-        <!-- laser -->
-        <link
-            name="laser_link">
-            <inertial>
-                <origin
-                    xyz="0.00196458631046099 -3.57895428399795E-06 0.00189816836722938"
-                    rpy="0 0 0" />
-                <mass
-                    value="0.0477519163775583" />
-                <inertia
-                    ixx="3.38461999766101E-05"
-                    ixy="-2.19897141950282E-09"
-                    ixz="1.07118468648131E-06"
-                    iyy="3.94150415881323E-05"
-                    iyz="6.83978165807776E-10"
-                    izz="5.60787042136426E-05" />
-            </inertial>
-            <visual>
-                <origin
-                    xyz="0 0 0"
-                    rpy="0 3.14159265358979 0" />
-                <geometry>
-                    <mesh
-                        filename="package://turn_on_32chassis/urdf/meshes/mid-360-asm.stl" />
-                </geometry>
-                <material
-                    name="">
-                    <color
-                        rgba="0.376470588235294 0.376470588235294 0.376470588235294 1" />
-                </material>
-            </visual>
-            <collision>
-                <origin
-                    xyz="0 0 0"
-                    rpy="0 3.14159265358979 0" />
-                <geometry>
-                    <mesh
-                        filename="package://turn_on_32chassis/urdf/meshes/mid-360-asm.stl" />
-                </geometry>
-            </collision>
-        </link>
-        <joint
-            name="laser_joint"
-            type="fixed">
-            <origin
-                xyz="0.0316310367407428 9.05810809801877E-05 0.115"
-                rpy="0 0 0" />
-            <parent
-                link="base_link" />
-            <child
-                link="laser_link" />
-            <axis
-                xyz="0 0 0" />
-        </joint>
-        <link
-            name="controller_link">
-            <inertial>
-                <origin
-                    xyz="-0.0178772421800459 0.0389174701067245 0.0213653101693057"
-                    rpy="0 0 0" />
-                <mass
-                    value="0.0391683061674007" />
-                <inertia
-                    ixx="2.20183096868336E-05"
-                    ixy="1.2570811872774E-06"
-                    ixz="1.53420711428651E-09"
-                    iyy="2.40630534171015E-05"
-                    iyz="2.27786586281681E-07"
-                    izz="4.51084285172614E-05" />
-            </inertial>
-            <visual>
-                <origin
-                    xyz="0 0 0"
-                    rpy="0 0 0" />
-                <geometry>
-                    <mesh
-                        filename="package://turn_on_32chassis/urdf/meshes/mini_4wd_robot_meshes/controller_link.STL" />
-                </geometry>
-                <material
-                    name="">
-                    <color
-                        rgba="1 1 1 1" />
-                </material>
-            </visual>
-            <collision>
-                <origin
-                    xyz="0 0 0"
-                    rpy="0 0 0" />
-                <geometry>
-                    <mesh
-                        filename="package://turn_on_32chassis/urdf/meshes/mini_4wd_robot_meshes/controller_link.STL" />
-                </geometry>
-            </collision>
-        </link>
-        <joint
-            name="controller_joint"
-            type="fixed">
-            <origin
-                xyz="-0.0556343132168706 -0.0407821141826353 0.0519999999999999"
-                rpy="0 0 0" />
-            <parent
-                link="base_link" />
-            <child
-                link="controller_link" />
-            <axis
-                xyz="0 0 0" />
-        </joint>
-        <!-- 深度相机传感器 -->
-        <!-- <link
-            name="camera_link">
-            <inertial>
-                <origin
-                    xyz="3.50190324967248E-07 9.10362268407238E-08 1.07624234177428E-07"
-                    rpy="0 0 0" />
-                <mass
-                    value="0.0559842512080236" />
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